Commit message: I have added a new test branch, please do the experimental changes in this only

File: src/robovacuum_description/urdf/robovacuum.urdf.xacro (robot description, xacro)
@@ -3,90 +3,18 @@
   <!-- Include ros2_control Plugins -->
   <xacro:include filename="$(find robovacuum_description)/urdf/robovacuum_ros2_control.xacro" />
-  <link name="base_footprint"/>
-  <link name="base_link">
-    <inertial>
-      <origin xyz="0 0 0.04" rpy="0.0 0.25 0.3" />
-      <mass value="8.2573504e-01"/>
-      <inertia ixx="2.2124416e-02" ixy="-1.2294101e-04" ixz="3.4938785e-04"
-               iyy="2.1193702e-02" iyz="-5.0120904e-05"
-               izz="2.0064271e-02" />
-    </inertial>
-  </link>
-  <joint name="base_joint" type="fixed">
-    <parent link="base_footprint"/>
-    <child link="base_link" />
-    <origin xyz="0 0 0.033" rpy="0 0 0"/>
+  <link name="base_link"/>
+  <link name="wheel_left_link"/>
+  <link name="wheel_right_link"/>
+  <joint name="wheel_left_joint" type="continuous">
+    <parent link="base_link"/>
+    <child link="wheel_left_link"/>
+    <origin xyz="0 0.2 0" rpy="0 0 0"/>
+    <axis xyz="0 1 0"/>
   </joint>
-  <link name="wheel_right_link">
-    <inertial>
-      <origin xyz="0 -0.014 0" rpy="0 0 0" />
-      <mass value="0.0530086090966721" />
-      <inertia ixx="1.88176298336665E-05" ixy="-4.8444933029987E-10" ixz="1.88163708851143E-08"
-               iyy="3.11510738647764E-05" iyz="-6.93560663069607E-11"
-               izz="1.8801969558182E-05" />
-    </inertial>
-  </link>
   <joint name="wheel_right_joint" type="continuous">
-    <origin xyz="0 -0.0701101849418637 0" rpy="0 0 0" />
-    <parent link="base_link" />
-    <child link="wheel_right_link" />
-    <axis xyz="0 1 0" />
-  </joint>
-  <link name="wheel_left_link">
-    <inertial>
-      <origin xyz="0 0.014 0" rpy="0 0 0" />
-      <mass value="0.0530086043217644" />
-      <inertia ixx="1.8792911368909E-05" ixy="3.31256392204584E-10" ixz="-1.14082001662767E-08"
-               iyy="3.11510738759073E-05" iyz="-3.60499245082192E-10"
-               izz="1.88266886146847E-05" />
-    </inertial>
-  </link>
-  <joint name="wheel_left_joint" type="continuous">
-    <origin xyz="0 0.0701101849418642 0" rpy="0 0 0" />
-    <parent link="base_link" />
-    <child link="wheel_left_link" />
-    <axis xyz="0 1 0" />
-  </joint>
-  <link name="caster_front_link">
-    <inertial>
-      <origin xyz="3.89968128948481E-07 2.40073004698083E-07 0.00219173397061506" rpy="0 0 0" />
-      <mass value="1.44379265037903E-06" />
-      <inertia ixx="7.23075276010246E-11" ixy="-6.10956883467859E-16" ixz="2.22849693525031E-15"
-               iyy="3.8713793085917E-11" iyz="2.93909858781952E-15"
-               izz="1.00967486676306E-10" />
-    </inertial>
-  </link>
-  <joint name="caster_front_joint" type="fixed">
-    <origin xyz="0.04755 0 -0.0275" rpy="0 0 0" />
-    <parent link="base_link" />
-    <child link="caster_front_link" />
-  </joint>
-  <link name="caster_rear_link">
-    <inertial>
-      <origin xyz="3.8996812895542E-07 2.40073004698083E-07 0.00219173397061509" rpy="0 0 0" />
-      <mass value="1.44379265037902E-06" />
-      <inertia ixx="7.23075276010246E-11" ixy="-6.10956872363424E-16" ixz="2.22849693527207E-15"
-               iyy="3.87137930859167E-11" iyz="2.939098587861E-15"
-               izz="1.00967486676306E-10" />
-    </inertial>
-  </link>
-  <joint name="caster_rear_joint" type="fixed">
-    <origin xyz="-0.04755 0 -0.0275" rpy="0 0 0" />
-    <parent link="base_link" />
-    <child link="caster_rear_link" />
-  </joint>
-  <link name="imu_link">
-    <inertial>
-      <origin xyz="-0.00552433659106688 0.000168210391520346 0.000514000497342681" rpy="0 0 0" />
-      <mass value="0.000528415362211671" />
-      <inertia ixx="1.46176048428261E-08" ixy="1.40015117949421E-10" ixz="-1.99633872937403E-12"
-               iyy="8.59662482954888E-09" iyz="7.52375112767959E-12"
-               izz="2.30279421279312E-08" />
-    </inertial>
-  </link>
-  <joint name="imu_joint" type="fixed">
-    <origin xyz="0 0 0.0698986241758014" rpy="0 0 0" />
-    <parent link="base_link" />
-    <child link="imu_link" />
+    <parent link="base_link"/>
+    <child link="wheel_right_link"/>
+    <origin xyz="0 -0.2 0" rpy="0 0 0"/>
+    <axis xyz="0 1 0"/>
   </joint>
 </robot>

File: src/robovacuum_description/urdf/robovacuum_ros2_control.xacro (robot description, xacro)
@@ -5,5 +5,5 @@
             <hardware>
                 <plugin>robovacuum_firmware/RobovacuumInterface</plugin>
-                <param name="port">/dev/ttyUSB0</param>
+                <param name="port">/dev/ttyACM0</param>
             </hardware>
         <!-- ros2_control Common Interfaces -->

Commit message: Starting with the simulation part also

File: src/robovacuum_description/urdf/robovacuum.urdf.xacro (robot description, xacro)
@@ -3,18 +3,105 @@
   <!-- Include ros2_control Plugins -->
   <xacro:include filename="$(find robovacuum_description)/urdf/robovacuum_ros2_control.xacro" />
-  <link name="base_link"/>
-  <link name="wheel_left_link"/>
-  <link name="wheel_right_link"/>
+  <xacro:include filename="$(find robovacuum_description)/urdf/inertial_macros.xacro" />
+  <material name="white">
+    <color rgba="1 1 1 1"/>
+  </material>
+  <material name="orange">
+    <color rgba="1 0.3 0.1 1"/>
+  </material>
+  <material name="blue">
+    <color rgba="0.2 0.2 1 1"/>
+  </material>
+  <material name="black">
+    <color rgba="0 0 0 1"/>
+  </material>
+  <link name="base_link"/>  <!--generally in the center of differential drive wheel-->
+  <link name="base_footprint">
+    <visual>
+      <origin xyz="-0.15 0 0"/>
+      <geometry>
+        <box size="0.3 0.4 0.05"/>
+      </geometry>
+      <material name="white"/>
+    </visual>
+    <collision>
+      <origin xyz="-0.15 0 0"/>
+      <geometry>
+        <box size="0.3 0.4 0.05"/>
+      </geometry>
+    </collision>
+    <xacro:inertial_box mass="10" x="0.3" y="0.4" z="0.05">
+      <origin xyz="-0.15 0 0" rpy="0 0 0"/>
+    </xacro:inertial_box>
+  </link>
+  <link name="wheel_left_link">
+    <visual>
+      <geometry>
+        <cylinder radius="0.1" length="0.05"/>
+      </geometry>
+      <material name="blue"/>
+    </visual>
+    <collision>
+      <geometry>
+        <cylinder radius="0.1" length="0.05"/>
+      </geometry>
+    </collision>
+    <xacro:inertial_cylinder mass="1.0" length="0.05" radius="0.1">
+      <origin xyz="0 0 0" rpy="0 0 0"/>
+    </xacro:inertial_cylinder>
+  </link>
+  <link name="wheel_right_link">
+    <visual>
+      <geometry>
+        <cylinder radius="0.1" length="0.05"/>
+      </geometry>
+      <material name="blue"/>
+    </visual>
+    <collision>
+      <geometry>
+        <cylinder radius="0.1" length="0.05"/>
+      </geometry>
+    </collision>
+    <xacro:inertial_cylinder mass="1.0" length="0.05" radius="0.1">
+      <origin xyz="0 0 0" rpy="0 0 0"/>
+    </xacro:inertial_cylinder>
+  </link>
+  <link name="caster_wheel">
+    <visual>
+      <geometry>
+        <sphere radius="0.05"/>
+      </geometry>
+      <material name="black"/>
+    </visual>
+    <collision>
+      <geometry>
+        <sphere radius="0.05"/>
+      </geometry>
+    </collision>
+    <xacro:inertial_sphere mass="0.1" radius="0.05">
+      <origin xyz="0 0 0" rpy="0 0 0"/>
+    </xacro:inertial_sphere>
+  </link>
+  <joint name="base_joint" type="fixed">
+    <parent link="base_link"/>
+    <child link="base_footprint"/>
+    <origin xyz="0.1 0 0"/>
+  </joint>
   <joint name="wheel_left_joint" type="continuous">
     <parent link="base_link"/>
     <child link="wheel_left_link"/>
-    <origin xyz="0 0.2 0" rpy="0 0 0"/>
-    <axis xyz="0 1 0"/>
+    <origin xyz="0 0.2 0" rpy="-${pi/2} 0 0"/>
+    <axis xyz="0 0 1"/>
   </joint>
   <joint name="wheel_right_joint" type="continuous">
     <parent link="base_link"/>
     <child link="wheel_right_link"/>
-    <origin xyz="0 -0.2 0" rpy="0 0 0"/>
-    <axis xyz="0 1 0"/>
+    <origin xyz="0 -0.2 0" rpy="${pi/2} 0 0"/>
+    <axis xyz="0 0 -1"/>
+  </joint>
+  <joint name="caster_wheel_joint" type="fixed">
+    <parent link="base_footprint"/>
+    <child link="caster_wheel"/>
+    <origin xyz="-0.24 0 0"/>
   </joint>
 </robot>

Commit message: changes in filmware files

File: src/robovacuum_description/urdf/robovacuum.urdf.xacro (robot description, xacro)
@@ -3,9 +3,9 @@
   <!-- Include ros2_control Plugins -->
   <xacro:include filename="$(find robovacuum_description)/urdf/robovacuum_ros2_control.xacro" />
-  <link name="base_link"/>
+  <link name="base_footprint"/>
   <link name="wheel_left_link"/>
   <link name="wheel_right_link"/>
   <joint name="wheel_left_joint" type="continuous">
-    <parent link="base_link"/>
+    <parent link="base_footprint"/>
     <child link="wheel_left_link"/>
     <origin xyz="0 0.2 0" rpy="0 0 0"/>
@@ -13,5 +13,5 @@
   </joint>
   <joint name="wheel_right_joint" type="continuous">
-    <parent link="base_link"/>
+    <parent link="base_footprint"/>
     <child link="wheel_right_link"/>
     <origin xyz="0 -0.2 0" rpy="0 0 0"/>

Commit message: changes in urdf according to the actual robot

File: src/robovacuum_description/urdf/robovacuum.urdf.xacro (robot description, xacro)
@@ -19,18 +19,18 @@
   <link name="base_footprint">
     <visual>
-      <origin xyz="-0.15 0 0"/>
+      <origin xyz="-0.2 0 0.05"/>
       <geometry>
-        <box size="0.3 0.4 0.05"/>
+        <box size="0.45 0.35 0.1"/>
       </geometry>
       <material name="white"/>
     </visual>
     <collision>
-      <origin xyz="-0.15 0 0"/>
+      <origin xyz="-0.2 0 0"/>
       <geometry>
-        <box size="0.3 0.4 0.05"/>
+        <box size="0.45 0.35 0.1"/>
       </geometry>
     </collision>
-    <xacro:inertial_box mass="10" x="0.3" y="0.4" z="0.05">
-      <origin xyz="-0.15 0 0" rpy="0 0 0"/>
+    <xacro:inertial_box mass="10" x="0.45" y="0.35" z="0.1">
+      <origin xyz="-0.2 0 0" rpy="0 0 0"/>
     </xacro:inertial_box>
   </link>
@@ -38,5 +38,5 @@
     <visual>
       <geometry>
-        <cylinder radius="0.1" length="0.05"/>
+        <cylinder radius="0.1" length="0.04"/>
       </geometry>
       <material name="blue"/>
@@ -44,8 +44,8 @@
     <collision>
       <geometry>
-        <cylinder radius="0.1" length="0.05"/>
+        <cylinder radius="0.1" length="0.04"/>
       </geometry>
     </collision>
-    <xacro:inertial_cylinder mass="1.0" length="0.05" radius="0.1">
+    <xacro:inertial_cylinder mass="1.0" length="0.04" radius="0.1">
       <origin xyz="0 0 0" rpy="0 0 0"/>
     </xacro:inertial_cylinder>
@@ -54,5 +54,5 @@
     <visual>
       <geometry>
-        <cylinder radius="0.1" length="0.05"/>
+        <cylinder radius="0.1" length="0.04"/>
       </geometry>
       <material name="blue"/>
@@ -60,8 +60,8 @@
     <collision>
       <geometry>
-        <cylinder radius="0.1" length="0.05"/>
+        <cylinder radius="0.1" length="0.04"/>
       </geometry>
     </collision>
-    <xacro:inertial_cylinder mass="1.0" length="0.05" radius="0.1">
+    <xacro:inertial_cylinder mass="1.0" length="0.04" radius="0.1">
       <origin xyz="0 0 0" rpy="0 0 0"/>
     </xacro:inertial_cylinder>
@@ -70,5 +70,5 @@
     <visual>
       <geometry>
-        <sphere radius="0.05"/>
+        <sphere radius="0.01"/>
       </geometry>
       <material name="black"/>
@@ -76,8 +76,8 @@
     <collision>
       <geometry>
-        <sphere radius="0.05"/>
+        <sphere radius="0.02"/>
       </geometry>
     </collision>
-    <xacro:inertial_sphere mass="0.1" radius="0.05">
+    <xacro:inertial_sphere mass="0.1" radius="0.01">
       <origin xyz="0 0 0" rpy="0 0 0"/>
     </xacro:inertial_sphere>
@@ -86,10 +86,10 @@
     <parent link="base_link"/>
     <child link="base_footprint"/>
-    <origin xyz="0.1 0 0"/>
+    <origin xyz="0.2 0 0"/>
   </joint>
   <joint name="wheel_left_joint" type="continuous">
     <parent link="base_link"/>
     <child link="wheel_left_link"/>
-    <origin xyz="0 0.2 0" rpy="-${pi/2} 0 0"/>
+    <origin xyz="0 0.175 0.05" rpy="-${pi/2} 0 0"/>
     <axis xyz="0 0 1"/>
   </joint>
@@ -97,5 +97,5 @@
     <parent link="base_link"/>
     <child link="wheel_right_link"/>
-    <origin xyz="0 -0.2 0" rpy="${pi/2} 0 0"/>
+    <origin xyz="0 -0.175 0.05" rpy="${pi/2} 0 0"/>
     <axis xyz="0 0 -1"/>
   </joint>
@@ -103,5 +103,5 @@
     <parent link="base_footprint"/>
     <child link="caster_wheel"/>
-    <origin xyz="-0.24 0 0"/>
+    <origin xyz="-0.43 0 0"/>
   </joint>
 </robot>

File: src/robovacuum_description/urdf/robovacuum_ros2_control.xacro (robot description, xacro)
@@ -5,5 +5,5 @@
             <hardware>
                 <plugin>robovacuum_firmware/RobovacuumInterface</plugin>
-                <param name="port">/dev/ttyACM0</param>
+                <param name="port">/dev/ttyACM1</param>
             </hardware>
         <!-- ros2_control Common Interfaces -->

Commit message: Simualation and Odometry features added

File: src/robovacuum_description/urdf/robovacuum.urdf.xacro (robot description, xacro)
@@ -1,7 +1,11 @@
 <?xml version="1.0"?>
 <robot name="robovacuum" xmlns:xacro="http://ros.org/wiki/xacro">
+  <xacro:arg name="is_ignition" default="true"/>
+  <xacro:arg name="is_sim" default="true"/>
   <!-- Include ros2_control Plugins -->
   <xacro:include filename="$(find robovacuum_description)/urdf/robovacuum_ros2_control.xacro" />
   <xacro:include filename="$(find robovacuum_description)/urdf/inertial_macros.xacro" />
+  <!--Inculude Gazebo Parameters-->
+  <xacro:include filename="$(find robovacuum_description)/urdf/robovacuum_gazebo.xacro" />
   <material name="white">
     <color rgba="1 1 1 1"/>
@@ -19,5 +23,5 @@
   <link name="base_footprint">
     <visual>
-      <origin xyz="-0.2 0 0.05"/>
+      <origin xyz="0.225 0 0.05"/>
       <geometry>
         <box size="0.45 0.35 0.1"/>
@@ -26,5 +30,5 @@
     </visual>
     <collision>
-      <origin xyz="-0.2 0 0"/>
+      <origin xyz="0.225 0 0.05"/>
       <geometry>
         <box size="0.45 0.35 0.1"/>
@@ -32,5 +36,5 @@
     </collision>
     <xacro:inertial_box mass="10" x="0.45" y="0.35" z="0.1">
-      <origin xyz="-0.2 0 0" rpy="0 0 0"/>
+      <origin xyz="0.225 0 0.05" rpy="0 0 0"/>
     </xacro:inertial_box>
   </link>
@@ -70,5 +74,5 @@
     <visual>
       <geometry>
-        <sphere radius="0.01"/>
+        <sphere radius="0.05"/>
       </geometry>
       <material name="black"/>
@@ -79,17 +83,33 @@
       </geometry>
     </collision>
-    <xacro:inertial_sphere mass="0.1" radius="0.01">
+    <xacro:inertial_sphere mass="0.1" radius="0.05">
       <origin xyz="0 0 0" rpy="0 0 0"/>
     </xacro:inertial_sphere>
   </link>
+  <link name="imu_link">
+  <visual>
+    <geometry>
+      <box size="0.025 0.02 0.003"/>  <!-- BNO055 dimensions: 25x20x3mm -->
+    </geometry>
+    <material name="blue"/>
+  </visual>
+  <collision>
+    <geometry>
+      <box size="0.025 0.02 0.003"/>
+    </geometry>
+  </collision>
+  <xacro:inertial_box mass="0.003" x="0.025" y="0.02" z="0.003">
+    <origin xyz="0 0 0" rpy="0 0 0"/>
+  </xacro:inertial_box>
+</link>
   <joint name="base_joint" type="fixed">
     <parent link="base_link"/>
     <child link="base_footprint"/>
-    <origin xyz="0.2 0 0"/>
+    <origin xyz="-0.2 0 -0.05"/>
   </joint>
   <joint name="wheel_left_joint" type="continuous">
     <parent link="base_link"/>
     <child link="wheel_left_link"/>
-    <origin xyz="0 0.175 0.05" rpy="-${pi/2} 0 0"/>
+    <origin xyz="0 0.175 0" rpy="-${pi/2} 0 0"/>
     <axis xyz="0 0 1"/>
   </joint>
@@ -97,5 +117,5 @@
     <parent link="base_link"/>
     <child link="wheel_right_link"/>
-    <origin xyz="0 -0.175 0.05" rpy="${pi/2} 0 0"/>
+    <origin xyz="0 -0.175 0" rpy="${pi/2} 0 0"/>
     <axis xyz="0 0 -1"/>
   </joint>
@@ -103,5 +123,10 @@
     <parent link="base_footprint"/>
     <child link="caster_wheel"/>
-    <origin xyz="-0.43 0 0"/>
+    <origin xyz="0.43 0 0"/>
+  </joint>
+  <joint name="imu_joint" type="fixed">
+    <parent link="base_footprint"/>
+    <child link="imu_link"/>
+    <origin xyz="0.225 0 0.1" rpy="0 0 0"/>
   </joint>
 </robot>

File: src/robovacuum_description/urdf/robovacuum_ros2_control.xacro (robot description, xacro)
@@ -2,9 +2,21 @@
 <robot xmlns:xacro="http://www.ros.org/wiki/xacro" name="robovacuum">
     <ros2_control name="RobotSystem" type="system">
+        <xacro:if value="$(arg is_ignition)">
+            <hardware>
+                <plugin>ign_ros2_control/IgnitionSystem</plugin>
+            </hardware>
+        </xacro:if>
+        <xacro:unless value="$(arg is_ignition)">
+            <hardware>
+                <plugin>gz_ros2_control/GazeboSimSystem</plugin>
+            </hardware>
+        </xacro:unless>
         <!-- ros2_control Real Robot -->
+         <xacro:unless value="$(arg is_sim)">
             <hardware>
                 <plugin>robovacuum_firmware/RobovacuumInterface</plugin>
                 <param name="port">/dev/ttyACM1</param>
             </hardware>
+         </xacro:unless>
         <!-- ros2_control Common Interfaces -->
         <joint name="wheel_right_joint">
