Commit message: Final changes

File: src/robovacuum_description/urdf/robovacuum.urdf.xacro (robot description, xacro)
@@ -1,4 +1,5 @@
 <?xml version="1.0"?>
-<robot name="robovacuum" xmlns:xacro="http://ros.org/wiki/xacro">
+<robot name="robovacuum"
+  xmlns:xacro="http://ros.org/wiki/xacro">
   <xacro:arg name="is_ignition" default="true"/>
   <xacro:arg name="is_sim" default="true"/>
@@ -20,5 +21,6 @@
     <color rgba="0 0 0 1"/>
   </material>
-  <link name="base_link"/>  <!--generally in the center of differential drive wheel-->
+  <link name="base_link"/>
+  <!--generally in the center of differential drive wheel-->
   <link name="base_footprint">
     <visual>
@@ -88,19 +90,41 @@
   </link>
   <link name="imu_link">
-  <visual>
-    <geometry>
-      <box size="0.025 0.02 0.003"/>  <!-- BNO055 dimensions: 25x20x3mm -->
-    </geometry>
-    <material name="blue"/>
-  </visual>
-  <collision>
-    <geometry>
-      <box size="0.025 0.02 0.003"/>
-    </geometry>
-  </collision>
-  <xacro:inertial_box mass="0.003" x="0.025" y="0.02" z="0.003">
-    <origin xyz="0 0 0" rpy="0 0 0"/>
-  </xacro:inertial_box>
-</link>
+    <visual>
+      <geometry>
+        <box size="0.025 0.02 0.003"/>
+        <!-- BNO055 dimensions: 25x20x3mm -->
+      </geometry>
+      <material name="blue"/>
+    </visual>
+    <collision>
+      <geometry>
+        <box size="0.025 0.02 0.003"/>
+      </geometry>
+    </collision>
+    <xacro:inertial_box mass="0.003" x="0.025" y="0.02" z="0.003">
+      <origin xyz="0 0 0" rpy="0 0 0"/>
+    </xacro:inertial_box>
+  </link>
+  <!-- ============ CAMERA LINK ============ -->
+  <link name="camera_link">
+    <visual>
+      <geometry>
+        <box size="0.075 0.025 0.027"/>
+        <!-- Kinect v2 dimensions -->
+      </geometry>
+      <material name="black"/>
+      <origin xyz="0 0 0" rpy="0 0 0"/>
+    </visual>
+    <collision>
+      <geometry>
+        <box size="0.075 0.025 0.027"/>
+      </geometry>
+      <origin xyz="0 0 0" rpy="0 0 0"/>
+    </collision>
+    <inertial>
+      <mass value="0.5"/>
+      <inertia ixx="0.001" ixy="0" ixz="0" iyy="0.001" iyz="0" izz="0.001"/>
+    </inertial>
+  </link>
   <joint name="base_joint" type="fixed">
     <parent link="base_link"/>
@@ -130,3 +154,17 @@
     <origin xyz="0.225 0 0.1" rpy="0 0 0"/>
   </joint>
+  <joint name="camera_joint" type="fixed">
+    <parent link="base_footprint"/>
+    <child link="camera_link"/>
+    <origin xyz="0.2 0 0.15" rpy="0 0.3 0"/>
+    <!-- 0.3 rad tilt = ~17 degrees down to see floor ahead -->
+  </joint>
+  <!-- Camera optical frame (required for image processing) -->
+  <link name="camera_depth_frame"/>
+  <joint name="camera_depth_joint" type="fixed">
+    <parent link="camera_link"/>
+    <child link="camera_depth_frame"/>
+    <origin xyz="0 0 0" rpy="-1.5708 0 -1.5708"/>
+    <!-- Rotation to align with ROS camera conventions -->
+  </joint>
 </robot>

File: src/robovacuum_description/urdf/robovacuum_gazebo.xacro (robot description, xacro)
@@ -1,4 +1,5 @@
 <?xml version="1.0"?>
-<robot name="bumperbot" xmlns:xacro="http://ros.org/wiki/xacro">
+<robot name="bumperbot"
+  xmlns:xacro="http://ros.org/wiki/xacro">
   <!-- Wheels -->
   <gazebo reference="wheel_left_link">
@@ -47,50 +48,81 @@
   <gazebo reference="imu_link">
     <sensor name="imu" type="imu">
-        <always_on>true</always_on>
-        <update_rate>100</update_rate>
-        <gz_frame_id>imu_link</gz_frame_id>
-        <topic>imu</topic>
-        <imu>
-          <angular_velocity>
-            <x>
-              <noise type="gaussian">
-                <mean>0.0</mean>
-                <stddev>2e-4</stddev>
-              </noise>
-            </x>
-            <y>
-              <noise type="gaussian">
-                <mean>0.0</mean>
-                <stddev>2e-4</stddev>
-              </noise>
-            </y>
-            <z>
-              <noise type="gaussian">
-                <mean>0.0</mean>
-                <stddev>2e-4</stddev>
-              </noise>
-            </z>
-          </angular_velocity>
-          <linear_acceleration>
-            <x>
-              <noise type="gaussian">
-                <mean>0.0</mean>
-                <stddev>1.7e-2</stddev>
-              </noise>
-            </x>
-            <y>
-              <noise type="gaussian">
-                <mean>0.0</mean>
-                <stddev>1.7e-2</stddev>
-              </noise>
-            </y>
-            <z>
-              <noise type="gaussian">
-                <mean>0.0</mean>
-                <stddev>1.7e-2</stddev>
-              </noise>
-            </z>
-          </linear_acceleration>
-        </imu>
+      <always_on>true</always_on>
+      <update_rate>100</update_rate>
+      <gz_frame_id>imu_link</gz_frame_id>
+      <topic>imu</topic>
+      <imu>
+        <angular_velocity>
+          <x>
+            <noise type="gaussian">
+              <mean>0.0</mean>
+              <stddev>2e-4</stddev>
+            </noise>
+          </x>
+          <y>
+            <noise type="gaussian">
+              <mean>0.0</mean>
+              <stddev>2e-4</stddev>
+            </noise>
+          </y>
+          <z>
+            <noise type="gaussian">
+              <mean>0.0</mean>
+              <stddev>2e-4</stddev>
+            </noise>
+          </z>
+        </angular_velocity>
+        <linear_acceleration>
+          <x>
+            <noise type="gaussian">
+              <mean>0.0</mean>
+              <stddev>1.7e-2</stddev>
+            </noise>
+          </x>
+          <y>
+            <noise type="gaussian">
+              <mean>0.0</mean>
+              <stddev>1.7e-2</stddev>
+            </noise>
+          </y>
+          <z>
+            <noise type="gaussian">
+              <mean>0.0</mean>
+              <stddev>1.7e-2</stddev>
+            </noise>
+          </z>
+        </linear_acceleration>
+      </imu>
+    </sensor>
+  </gazebo>
+  <!-- ============ CAMERA SENSOR ============ -->
+  <gazebo reference="camera_link">
+    <sensor name="depth_camera" type="depth_camera">
+      <camera>
+        <horizontal_fov>1.047</horizontal_fov>        <!-- 60 degrees -->
+        <image>
+          <width>512</width>
+          <height>424</height>
+        </image>
+        <clip>
+          <near>0.1</near>
+          <far>10.0</far>
+        </clip>
+      </camera>
+      <always_on>true</always_on>
+      <update_rate>30</update_rate>      <!-- 30 Hz update rate -->
+      <visualize>true</visualize>
+      <plugin name="camera_controller" filename="libgazebo_ros_depth_camera.so">
+        <ros>
+          <argument>~/image_raw:=camera/color/image_raw</argument>
+          <argument>~/image_depth:=camera/depth/image_raw</argument>
+          <argument>~/camera_info:=camera/camera_info</argument>
+          <argument>~/depth_image_raw:=camera/depth/image_raw</argument>
+          <argument>~/depth_camera_info:=camera/depth/camera_info</argument>
+          <argument>~/points:=camera/depth/points</argument>
+        </ros>
+        <camera_name>camera</camera_name>
+        <frame_name>camera_depth_frame</frame_name>
+      </plugin>
     </sensor>
   </gazebo>
